Commit message: Add ik stuff

File: catkin_ws/src/baymax_visualization/urdf/dofbot.urdf (robot description, URDF)
Before this commit: robot dofbot, 6 links, 5 joints
Joints:
- joint joint2: axis 0 0 1 -> 0 -1 0; origin xyz=0 -0.00031873 0.04145 rpy=0 1.5708 0 -> xyz=0 -0.00031873 0.04145 rpy=0 0 0
- joint joint3: axis 0 0 1 -> 0 -1 0; origin xyz=-0.08285 0 0 rpy=0 0 0 -> xyz=0 0 0.08285 rpy=0 0 0
- joint joint4: axis 0 0 1 -> 0 -1 0; origin xyz=-0.08285 0 0 rpy=0 0 0.0083081 -> xyz=0 0 0.08285 rpy=0 0 0
- joint joint5: origin xyz=-0.07385 -0.001 0 rpy=0 -1.57 0 -> xyz=0 0 0.07385 rpy=0 0 0

Commit message: cleaned up urdf, added camera frame, naive fk and marker images

File: catkin_ws/src/baymax_visualization/urdf/dofbot.urdf (robot description, URDF)
Before this commit: robot dofbot, 6 links, 5 joints
Links:
- added link link_cam
Joints:
- added joint cam: type fixed, parent link4, child link_cam, origin xyz=-0.072 -0.049 0 rpy=0 -1.5708 0
- joint joint1: origin xyz=0 0 0.06605 rpy=-0.010805 0 0 -> xyz=0 0 0.06605 rpy=0 0 0
- joint joint2: origin xyz=0 -0.00031873 0.04145 rpy=0 1.5708 0 -> xyz=0 0 0.04145 rpy=0 1.5708 0
- joint joint4: origin xyz=-0.08285 0 0 rpy=0 0 0.0083081 -> xyz=-0.08285 0 0 rpy=0 0 0
- joint joint5: origin xyz=-0.07385 -0.001 0 rpy=0 -1.57 0 -> xyz=-0.07385 0 0 rpy=0 -1.5708 0

Commit message: added tool frame to urdf, vision uses color segmentation)

File: catkin_ws/src/baymax_visualization/urdf/dofbot.urdf (robot description, URDF)
Before this commit: robot dofbot, 7 links, 6 joints
Links:
- added link link_tool
Joints:
- added joint tool: type fixed, parent link5, child link_tool, origin xyz=0 0 0.09 rpy=0 0 0

Commit message: new state messages, vision broadcasts markers for visualization, pid back in simulation package, other misc

File: catkin_ws/src/baymax_visualization/urdf/dofbot.urdf (robot description, URDF)
Before this commit: robot dofbot, 8 links, 7 joints
Joints:
- joint tool: origin xyz=0 0 0.09 rpy=0 0 0 -> xyz=0 0 0.11 rpy=0 0 0
